File: Hardware/ShieldPCB/NicoLase Arduino Shield.brd (EAGLE design)
At the start: 54.3 x 62.2 mm, 19 parts, among them IC1 4050D, J1 ARDUINO_R3_SHIELD, U1 7432SE

Commit message: Fixed error in trace of MASTERFIRE on PCB.  .brd file updated.  Removed Gerber files as they are incorrect, but not able to re-generate at this time.
Routing:
- net SLAVEFIRE: track 42.1 -> 46.0 mm
Changed lines of the file:
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@@
 <?xml version="1.0" encoding="utf-8"?>
 <!DOCTYPE eagle SYSTEM "eagle.dtd">
-<eagle version="7.4.0">
+<eagle version="8.0.0">
 <drawing>
 <settings>
@@
 <wire x1="21.59" y1="25.4" x2="21.59" y2="26.67" width="0.4064" layer="1"/>
 <wire x1="21.59" y1="26.67" x2="20.32" y2="27.94" width="0.4064" layer="1"/>
-<wire x1="20.32" y1="27.94" x2="17.78" y2="27.94" width="0.4064" layer="1"/>
+<wire x1="17.78" y1="27.94" x2="20.32" y2="27.94" width="0.4064" layer="1"/>
 <wire x1="27.62" y1="25.4" x2="30.48" y2="25.4" width="0.4064" layer="1"/>
 <contactref element="R5" pad="2"/>
@@
 <wire x1="29.845" y1="36.0934" x2="29.845" y2="33.655" width="0.4064" layer="1"/>
 <wire x1="29.845" y1="33.655" x2="30.48" y2="33.02" width="0.4064" layer="1"/>
-<wire x1="15.24" y1="29.21" x2="17.78" y2="27.94" width="0" layer="19" extent="1-1"/>
 <wire x1="30.48" y1="25.4" x2="33.02" y2="27.94" width="0.4064" layer="1"/>
 <wire x1="33.02" y1="27.94" x2="38.1" y2="27.94" width="0.4064" layer="1"/>
@@
 <wire x1="38.1" y1="31.75" x2="30.48" y2="31.75" width="0.4064" layer="1"/>
 <wire x1="30.48" y1="31.75" x2="30.48" y2="33.02" width="0.4064" layer="1"/>
+<wire x1="15.24" y1="29.21" x2="17.78" y2="29.21" width="0.4064" layer="1"/>
+<wire x1="17.78" y1="29.21" x2="17.78" y2="27.94" width="0.4064" layer="1"/>
 </signal>
 <signal name="N$2">
@@
 <wire x1="32.385" y1="33.655" x2="33.02" y2="33.02" width="0.4064" layer="1"/>
 <via x="33.02" y="33.02" extent="1-16" drill="0.6" shape="square"/>
-<wire x1="33.02" y1="33.02" x2="25.4" y2="33.02" width="0.4064" layer="16"/>
-<wire x1="25.4" y1="33.02" x2="24.13" y2="31.75" width="0.4064" layer="16"/>
+<wire x1="24.13" y1="31.75" x2="25.4" y2="33.02" width="0.4064" layer="16"/>
 <via x="24.13" y="31.75" extent="1-16" drill="0.6" shape="square"/>
 <wire x1="24.13" y1="31.75" x2="24.13" y2="27.64" width="0.4064" layer="1"/>
 <wire x1="24.13" y1="27.64" x2="25.72" y2="26.05" width="0.4064" layer="1"/>
 <wire x1="32.385" y1="33.655" x2="32.385" y2="36.0934" width="0.4064" layer="1"/>
+<wire x1="25.4" y1="33.02" x2="33.02" y2="33.02" width="0.4064" layer="16"/>
 </signal>
 <signal name="N$11">
